File: V1.5.kicad_pcb (KiCad board)
At the start: 2 copper layers, 28.6 x 24.4 mm, 18 parts, among them J1 Conn_01x08_Male, Q1 BC557, Q2 BUZ11, U1 LM78M05_TO252

Commit message: add info of v1.5.
Other:
- board text added: "V1.5 add diode D2, LED, 78M05, capacitors, holes for wires"
Changed lines of the file:
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@@
+    (effects (font (size 1 1) (thickness 0.15)))
+  )
+  (gr_text "V1.5\n\nadd diode D2, LED, 78M05, capacitors, holes for wires" (at 202.946 92.583) (layer "Edge.Cuts")
     (effects (font (size 1 1) (thickness 0.15)))
   )

Commit message: preparing for next drawing
Parts:
- removed C1: 2.2uF25V, Capacitor_SMD:CP_Elec_4x5.4
- removed C2, C3: 0.1uf, Capacitor_SMD:C_1206_3216Metric_Pad1.33x1.80mm_HandSolder
- removed D1: 1N4007, Diode_SMD:D_SMA
- removed D2: D_Schottky, Diode_THT:D_DO-27_P12.70mm_Horizontal
- removed D3: LED, LED_SMD:LED_1206_3216Metric_Pad1.42x1.75mm_HandSolder
- removed G***: LOGO, Logo:Logo
- removed J1: Conn_01x08_Male, Connector_PinHeader_2.54mm:PinHeader_1x08_P2.54mm_Vertical
- removed JP1: SolderJumper_2_Open, Jumper:SolderJumper-2_P1.3mm_Open_RoundedPad1.0x1.5mm
- removed Q1: BC557, Package_TO_SOT_THT:TO-92_Inline
- removed Q2: BUZ11, Package_TO_SOT_THT:TO-220F-3_Horizontal_TabDown
- removed R1: 220K, Resistor_SMD:R_1206_3216Metric_Pad1.30x1.75mm_HandSolder
- removed R2: 330K, Resistor_SMD:R_1206_3216Metric_Pad1.30x1.75mm_HandSolder
- removed R3, R4, R5: 10K, Resistor_SMD:R_1206_3216Metric_Pad1.30x1.75mm_HandSolder
- removed R6: 330, Resistor_SMD:R_1206_3216Metric_Pad1.30x1.75mm_HandSolder
- removed U1: LM78M05_TO252, Package_TO_SOT_SMD:TO-252-2
Routing:
- net /OUT-: track 57.4 -> 0.00 mm, vias 2 -> 0
- net /IN+: track 56.1 -> 0.00 mm
- net Net-(D1-Pad2): track 54.7 -> 0.00 mm, vias 1 -> 0
- net /LED+: track 33.6 -> 0.00 mm
- net /SW1: track 33.1 -> 0.00 mm
- net /IN-: track 31.8 -> 0.00 mm, vias 1 -> 0
- net Net-(Q1-Pad1): track 27.8 -> 0.00 mm
- net Net-(C3-Pad2): track 27.0 -> 0.00 mm, vias 3 -> 0
- net /SW2: track 13.2 -> 0.00 mm
- net Net-(Q1-Pad2): track 5.68 -> 0.00 mm
- net Net-(D3-Pad2): track 2.85 -> 0.00 mm
- removed copper zone on B.Cu, net (none)
- removed copper zone on F.Cu, net (none)
Other:
- board outline removed
- board text removed: "L- L+ SW SW OUT- OUT+ IN- IN+"
- board text removed: "v1.5"
